File: boards/ram-prototype/column_select.kicad_sch (KiCad schematic)
At the start: 6 parts, among them U1 74LVC1G04, U2 74LVC1G04

Commit message: Add initial changes to make logic close to final
Parts:
- added D10, D11, D12, D13, D14, D15, D16, D17, D18, D19, D20, D21, D22, D23, D24, D25, D26, D27, D28, D3, D4, D5, D6, D7, D8, D9: Red, symbol Device:LED_Small
- added R10, R11, R12, R13, R14, R15, R16, R17, R18, R19, R20, R21, R22, R23, R24, R25, R26, R27, R28, R3, R4, R5, R6, R7, R8, R9: 680R, symbol Device:R_Small
- added U10, U11, U12, U13, U14, U15, U16, U17, U18, U19, U20, U21, U22, U23, U24, U25, U26, U27, U28, U5, U6, U7, U8, U9: 74LVC1G08, symbol 74xGxx:74LVC1G08
- added U3, U4: 74LVC1G04, symbol 74xGxx:74LVC1G04
Connections:
- net COL_SEL_0: now also D13.2 (A), U13.4; no longer D1.2 (A), U1.4, U2.2
- net COL_SEL_1: now also D14.2 (A), U14.4; no longer D2.2 (A), U2.4
- net GND: now also R10.2, R11.2, R12.2, R13.2, R14.2, R15.2, R16.2, R17.2, R18.2, R19.2, R20.2, R21.2, R22.2, R23.2, R24.2, R25.2, R26.2, R27.2, R28.2, R3.2, R4.2, R5.2, R6.2, R7.2, R8.2, R9.2, U10.3 (GND), U11.3 (GND), U12.3 (GND), U13.3 (GND), U14.3 (GND), U15.3 (GND), U16.3 (GND), U17.3 (GND), U18.3 (GND), U19.3 (GND), U20.3 (GND), U21.3 (GND), U22.3 (GND), U23.3 (GND), U24.3 (GND), U25.3 (GND), U26.3 (GND), U27.3 (GND), U28.3 (GND), U3.3 (GND), U4.3 (GND), U5.3 (GND), U6.3 (GND), U7.3 (GND), U8.3 (GND), U9.3 (GND)
- net VCC: now also U10.5 (VCC), U11.5 (VCC), U12.5 (VCC), U13.5 (VCC), U14.5 (VCC), U15.5 (VCC), U16.5 (VCC), U17.5 (VCC), U18.5 (VCC), U19.5 (VCC), U20.5 (VCC), U21.5 (VCC), U22.5 (VCC), U23.5 (VCC), U24.5 (VCC), U25.5 (VCC), U26.5 (VCC), U27.5 (VCC), U28.5 (VCC), U3.5 (VCC), U4.5 (VCC), U5.5 (VCC), U6.5 (VCC), U7.5 (VCC), U8.5 (VCC), U9.5 (VCC)
- net A2 renamed A7
- net A7: now also U6.2, U8.2
- new net: D28.1 (K), R28.1
- new net: D15.1 (K), R15.1
- new net: D18.1 (K), R18.1
- new net: D24.1 (K), R24.1
- new net: D26.1 (K), R26.1
- new net: D9.1 (K), R9.1
- new net: D12.1 (K), R12.1
- new net: D8.1 (K), R8.1
- new net: D23.1 (K), R23.1
- new net: D4.2 (A), U10.1, U4.4, U9.1
- new net: D11.1 (K), R11.1
- new net: D13.1 (K), R13.1
- new net: D19.1 (K), R19.1
- new net: D2.2 (A), U2.4, U5.1, U6.1
- new net: D3.2 (A), U11.2, U3.4, U9.2
- new net: D14.1 (K), R14.1
- new net: D17.1 (K), R17.1
- new net: D7.1 (K), R7.1
- new net: D21.1 (K), R21.1
- new net: D4.1 (K), R4.1
- new net: D20.1 (K), R20.1
- new net: D1.2 (A), U1.4, U5.2, U7.2
- new net: D10.1 (K), R10.1
- new net: D6.1 (K), R6.1
- new net: D5.1 (K), R5.1
- new net: D22.1 (K), R22.1
- new net: D3.1 (K), R3.1
- new net: D27.1 (K), R27.1
- new net: D16.1 (K), R16.1
- new net: D25.1 (K), R25.1
- new net A10: U11.1, U12.1, U4.2
- new net A8: U2.2, U7.1, U8.1
- new net A9: U10.2, U12.2, U3.2
- new net COL_SEL_10: D23.2 (A), U23.4
- new net COL_SEL_11: D24.2 (A), U24.4
- new net COL_SEL_12: D25.2 (A), U25.4
- new net COL_SEL_13: D26.2 (A), U26.4
- new net COL_SEL_14: D27.2 (A), U27.4
- new net COL_SEL_15: D28.2 (A), U28.4
- new net COL_SEL_2: D15.2 (A), U15.4
- new net COL_SEL_3: D16.2 (A), U16.4
- new net COL_SEL_4: D17.2 (A), U17.4
- new net COL_SEL_5: D18.2 (A), U18.4
- new net COL_SEL_6: D19.2 (A), U19.4
- new net COL_SEL_7: D20.2 (A), U20.4
- new net COL_SEL_8: D21.2 (A), U21.4
- new net COL_SEL_9: D22.2 (A), U22.4
- new net GA0: D5.2 (A), U13.2, U17.2, U21.2, U25.2, U5.4
- new net GA1: D6.2 (A), U14.2, U18.2, U22.2, U26.2, U6.4
- new net GA2: D7.2 (A), U15.2, U19.2, U23.2, U27.2, U7.4
- new net GA3: D8.2 (A), U16.2, U20.2, U24.2, U28.2, U8.4
- new net GB0: D9.2 (A), U13.1, U14.1, U15.1, U16.1, U9.4
- new net GB1: D10.2 (A), U10.4, U17.1, U18.1, U19.1, U20.1
- new net GB2: D11.2 (A), U11.4, U21.1, U22.1, U23.1, U24.1
- new net GB3: D12.2 (A), U12.4, U25.1, U26.1, U27.1, U28.1
