File: boards/ram-prototype/ram.kicad_sch (KiCad schematic)
At the start: 48 parts, among them J1 SRAM_Bus, J2 DEC3_Unused, J3 Unused_COL_SEL, J4 DEC4_Unused

Commit message: Fix more issues
Connections:
- net D0: now also D18.2 (A), J1.6 (Pin_6); no longer D15.2 (A), J1.9 (Pin_9)
- net D1: now also D17.2 (A), J1.7 (Pin_7); no longer D14.2 (A), J1.10 (Pin_10)
- net D2: now also D16.2 (A), J1.8 (Pin_8); no longer D13.2 (A), J1.11 (Pin_11)
- net D3: now also D15.2 (A), J1.9 (Pin_9); no longer D12.2 (A), J1.12 (Pin_12)
- net D4: now also D14.2 (A), J1.10 (Pin_10); no longer D11.2 (A), J1.13 (Pin_13)
- net D5: now also D13.2 (A), J1.11 (Pin_11); no longer D10.2 (A), J1.14 (Pin_14)
- net D6: now also D12.2 (A), J1.12 (Pin_12); no longer D9.2 (A), J1.15 (Pin_15)
- net D7: now also D11.2 (A), J1.13 (Pin_13); no longer D8.2 (A), J1.16 (Pin_16)
- net nCE: now also D10.2 (A), J1.14 (Pin_14); no longer D18.2 (A), J1.6 (Pin_6)
- net nOE: now also D8.2 (A), J1.16 (Pin_16); no longer D16.2 (A), J1.8 (Pin_8)
- net nWE: now also D9.2 (A), J1.15 (Pin_15); no longer D17.2 (A), J1.7 (Pin_7)
