File: boards/ram-prototype/ram.kicad_pcb (KiCad board)
At the start: 4 copper layers, 173 x 118 mm, 611 parts, among them J1 PinHeader_1x24_P2.54mm_Vertic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, J2 PinHeader_1x04_P2.54mm_Vertic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, J3 PinHeader_1x14_P2.54mm_Vertic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, J4 PinHeader_2x08_P2.54mm_Vertic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, U1 DSBGA\-5_NumericPads, U10 DSBGA\-5_NumericPads, U100 DSBGA\-5_NumericPads, U101 DSBGA\-5_NumericPads, U102 DSBGA\-5_NumericPads, U103 DSBGA\-5_NumericPads, U104 DSBGA\-5_NumericPads, U105 DSBGA\-5_NumericPads, U106 DSBGA\-5_NumericPads, U107 DSBGA\-5_NumericPads, U108 DSBGA\-5_NumericPads, U109 DSBGA\-5_NumericPads, U11 DSBGA\-5_NumericPads, U110 DSBGA\-5_NumericPads, U111 DSBGA\-5_NumericPads, U112 DSBGA\-5_NumericPads, U113 DSBGA\-5_NumericPads, U114 DSBGA\-5_NumericPads, U115 DSBGA\-5_NumericPads, U116 DSBGA\-5_NumericPads, U117 DSBGA\-5_NumericPads, U118 DSBGA\-5_NumericPads, U119 DSBGA\-5_NumericPads, U12 DSBGA\-5_NumericPads, U120 DSBGA\-5_NumericPads, U121 DSBGA\-5_NumericPads, U122 DSBGA\-5_NumericPads, U123 DSBGA\-5_NumericPads, U124 DSBGA\-5_NumericPads, U125 DSBGA\-5_NumericPads, U126 DSBGA\-5_NumericPads, U127 DSBGA\-5_NumericPads, U128 DSBGA\-5_NumericPads, U129 DSBGA\-5_NumericPads, U13 DSBGA\-5_NumericPads, U130 DSBGA\-5_NumericPads, U131 DSBGA\-5_NumericPads, U132 DSBGA\-5_NumericPads, U133 DSBGA\-5_NumericPads, U134 DSBGA\-5_NumericPads, U135 DSBGA\-5_NumericPads, U136 DSBGA\-5_NumericPads, U137 DSBGA\-5_NumericPads, U138 DSBGA\-5_NumericPads, U139 DSBGA\-5_NumericPads, U14 DSBGA\-5_NumericPads, U140 DSBGA\-5_NumericPads, U141 DSBGA\-5_NumericPads, U142 DSBGA\-5_NumericPads, U143 DSBGA\-5_NumericPads, U144 DSBGA\-5_NumericPads, U145 DSBGA\-5_NumericPads, U146 DSBGA\-5_NumericPads, U147 DSBGA\-5_NumericPads, U148 DSBGA\-5_NumericPads, U149 DSBGA\-5_NumericPads, U15 DSBGA\-5_NumericPads, U150 DSBGA\-5_NumericPads, U151 DSBGA\-5_NumericPads, U152 DSBGA\-5_NumericPads, U153 DSBGA\-5_NumericPads, U154 DSBGA\-5_NumericPads, U155 DSBGA\-5_NumericPads, U156 DSBGA\-5_NumericPads, U157 DSBGA\-5_NumericPads, U158 DSBGA\-5_NumericPads, U159 DSBGA\-5_NumericPads, U16 DSBGA\-5_NumericPads, U160 DSBGA\-5_NumericPads, U161 DSBGA\-5_NumericPads, U162 DSBGA\-5_NumericPads, U163 DSBGA\-5_NumericPads, U164 DSBGA\-5_NumericPads, U165 DSBGA\-5_NumericPads, U166 DSBGA\-5_NumericPads, U167 DSBGA\-5_NumericPads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

Commit message: reorder connector control pins to nCE/nOE/nWE top-to-bottom
Move nCE to pin 8 (top), nOE to pin 7, nWE to pin 6 (bottom) on the
24-pin connector. Previous order was nCE/nWE/nOE which put nCE at the
bottom, making it harder for the autorouter to reach control_logic.

Post-routing: 3 errors (2 solder mask bridge), 3 warnings. The nCE
unconnected error from the previous run is eliminated.

Co-Authored-By: Claude Opus 4.6 (1M context) <noreply@anthropic.com>
Connections:
- D16 pad 2: /nOE -> /nCE
- D17 pad 2: /nWE -> /nOE
- D18 pad 2: /nCE -> /nWE
- J1 pad 6: /nCE -> /nWE
- J1 pad 7: /nWE -> /nOE
- J1 pad 8: /nOE -> /nCE
Changed lines of the file:
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@@
       (net 55 "/Column Select/A10"))
     (pad "6" thru_hole circle (at 0 12.7 180) (size 1.7 1.7) (drill 1) (layers *.Cu *.Mask) (remove_unused_layers no)
-      (net 102 "/nCE"))
-    (pad "7" thru_hole circle (at 0 15.24 180) (size 1.7 1.7) (drill 1) (layers *.Cu *.Mask) (remove_unused_layers no)
       (net 104 "/nWE"))
-    (pad "8" thru_hole circle (at 0 17.78 180) (size 1.7 1.7) (drill 1) (layers *.Cu *.Mask) (remove_unused_layers no)
+    (pad "7" thru_hole circle (at 0 15.24 180) (size 1.7 1.7) (drill 1) (layers *.Cu *.Mask) (remove_unused_layers no)
       (net 103 "/nOE"))
+    (pad "8" thru_hole circle (at 0 17.78 180) (size 1.7 1.7) (drill 1) (layers *.Cu *.Mask) (remove_unused_layers no)
+      (net 102 "/nCE"))
     (pad "9" thru_hole circle (at 0 20.32 180) (size 1.7 1.7) (drill 1) (layers *.Cu *.Mask) (remove_unused_layers no)
       (net 64 "/D0"))
@@
       (net 122 "Net-(D16-K)"))
     (pad "2" smd roundrect (at 0.485 0 180) (size 0.59 0.64) (layers "F.Cu" "F.Mask" "F.Paste") (roundrect_rratio 0.25)
-      (net 103 "/nOE"))
+      (net 102 "/nCE"))
     (embedded_fonts no)
     (model "${KICAD9_3DMODEL_DIR}/LED_SMD.3dshapes/LED_0402_1005Metric.step"
@@
       (net 123 "Net-(D17-K)"))
     (pad "2" smd roundrect (at 0.485 0 180) (size 0.59 0.64) (layers "F.Cu" "F.Mask" "F.Paste") (roundrect_rratio 0.25)
-      (net 104 "/nWE"))
+      (net 103 "/nOE"))
     (embedded_fonts no)
     (model "${KICAD9_3DMODEL_DIR}/LED_SMD.3dshapes/LED_0402_1005Metric.step"
@@
       (net 124 "Net-(D18-K)"))
     (pad "2" smd roundrect (at 0.485 0 180) (size 0.59 0.64) (layers "F.Cu" "F.Mask" "F.Paste") (roundrect_rratio 0.25)
-      (net 102 "/nCE"))
+      (net 104 "/nWE"))
     (embedded_fonts no)
     (model "${KICAD9_3DMODEL_DIR}/LED_SMD.3dshapes/LED_0402_1005Metric.step"
@@
   (segment (start 26.52 118.44) (end 26.82 118.74) (width 0.2) (layer "F.Cu") (net 55))
   (segment (start 26.82 118.74) (end 30.35 118.74) (width 0.2) (layer "F.Cu") (net 55))
-  (segment (start 20.0 114.8) (end 26.52 114.8) (width 0.2) (layer "F.Cu") (net 102))
+  (segment (start 20.0 114.8) (end 26.52 114.8) (width 0.2) (layer "F.Cu") (net 104))
   (segment (start 27.48 114.8) (end 28.35 114.8) (width 0.2) (layer "F.Cu") (net 124))
-  (segment (start 26.52 114.8) (end 26.52 115.9) (width 0.2) (layer "F.Cu") (net 102))
-  (segment (start 26.52 115.9) (end 26.82 116.2) (width 0.2) (layer "F.Cu") (net 102))
-  (segment (start 26.82 116.2) (end 30.35 116.2) (width 0.2) (layer "F.Cu") (net 102))
-  (segment (start 20.0 112.26) (end 26.52 112.26) (width 0.2) (layer "F.Cu") (net 104))
+  (segment (start 26.52 114.8) (end 26.52 115.9) (width 0.2) (layer "F.Cu") (net 104))
+  (segment (start 26.52 115.9) (end 26.82 116.2) (width 0.2) (layer "F.Cu") (net 104))
+  (segment (start 26.82 116.2) (end 30.35 116.2) (width 0.2) (layer "F.Cu") (net 104))
+  (segment (start 20.0 112.26) (end 26.52 112.26) (width 0.2) (layer "F.Cu") (net 103))
   (segment (start 27.48 112.26) (end 28.35 112.26) (width 0.2) (layer "F.Cu") (net 123))
-  (segment (start 26.52 112.26) (end 26.52 113.36) (width 0.2) (layer "F.Cu") (net 104))
-  (segment (start 26.52 113.36) (end 26.82 113.66) (width 0.2) (layer "F.Cu") (net 104))
-  (segment (start 26.82 113.66) (end 30.35 113.66) (width 0.2) (layer "F.Cu") (net 104))
-  (segment (start 20.0 109.72) (end 26.52 109.72) (width 0.2) (layer "F.Cu") (net 103))
+  (segment (start 26.52 112.26) (end 26.52 113.36) (width 0.2) (layer "F.Cu") (net 103))
+  (segment (start 26.52 113.36) (end 26.82 113.66) (width 0.2) (layer "F.Cu") (net 103))
+  (segment (start 26.82 113.66) (end 30.35 113.66) (width 0.2) (layer "F.Cu") (net 103))
+  (segment (start 20.0 109.72) (end 26.52 109.72) (width 0.2) (layer "F.Cu") (net 102))
   (segment (start 27.48 109.72) (end 28.35 109.72) (width 0.2) (layer "F.Cu") (net 122))
-  (segment (start 26.52 109.72) (end 26.52 110.82) (width 0.2) (layer "F.Cu") (net 103))
-  (segment (start 26.52 110.82) (end 26.82 111.12) (width 0.2) (layer "F.Cu") (net 103))
-  (segment (start 26.82 111.12) (end 30.35 111.12) (width 0.2) (layer "F.Cu") (net 103))
+  (segment (start 26.52 109.72) (end 26.52 110.82) (width 0.2) (layer "F.Cu") (net 102))
+  (segment (start 26.52 110.82) (end 26.82 111.12) (width 0.2) (layer "F.Cu") (net 102))
+  (segment (start 26.82 111.12) (end 30.35 111.12) (width 0.2) (layer "F.Cu") (net 102))
   (segment (start 20.0 107.18) (end 26.52 107.18) (width 0.2) (layer "F.Cu") (net 64))
   (segment (start 27.48 107.18) (end 28.35 107.18) (width 0.2) (layer "F.Cu") (net 121))
