File: boards/ram-prototype/power_supply.kicad_sch (KiCad schematic)
At the start: 19 parts, among them J1 PCIe_8pin, U1 TPS546D24A

Commit message: add manufacturing file generation and exclude connectors from BOM
- Add generate_manufacturing.py: gerbers, drill, BOM (with MPNs), and CPL for PCBWay
- Add in_bom parameter to SchematicBuilder.place_symbol() for native KiCad BOM exclusion
- Set in_bom=False on all 5 connectors (J1-J5) in generate_ram.py
- Regenerate schematics, PCB, and routed PCB

Co-Authored-By: Claude Opus 4.6 (1M context) <noreply@anthropic.com>
Parts:
- J1: now left out of the parts list
